Commit message: update

File: urdf_ex/urdf/gazebo.urdf.xacro (robot description, xacro)
@@ -76,5 +76,6 @@
         <clip>
           <near>0.05</near>
-          <far>3</far>
+          <far>10</far>
+          <!-- m 기준 카메라 멀리 보이기 -->
         </clip>
       </camera>

File: urdf_ex/urdf/test.urdf.xacro (robot description, xacro)
@@ -25,5 +25,6 @@
             <origin rpy="0 0 0" xyz="0 0 0"/>
             <geometry>
-                <box size="0.32 0.40 0.16"/>
+                <!-- <box size="0.32 0.40 0.16"/> -->
+                <box size="0.40 0.32 0.16"/>
             </geometry>
         </collision>
@@ -31,5 +32,5 @@
             <origin rpy="0 0 0" xyz="0 0 0"/>
             <geometry>
-                <box size="0.32 0.40 0.16"/>
+                <box size="0.40 0.32 0.16"/>
             </geometry>
             <material name="TEST_COL"/>
@@ -43,5 +44,5 @@
     <joint name="base_joint" type="fixed">
         <parent link="base_footprint"/>
-        <origin rpy="0 0 -1.57" xyz="0 0 0.11"/>
+        <origin rpy="0 0 0" xyz="0 0 0.11"/>
         <child link="base_link"/>
     </joint>
@@ -70,16 +71,17 @@
             <parent link="base_link"/>
             <child link="rear_caster_rotate_${prefix}"/>
-            <origin rpy="0 0 0" xyz="${dir*0.19} 0.17 -0.04"/>
+            <!-- <origin rpy="0 0 0" xyz="${dir*0.19} 0.17 -0.04"/> -->
+            <origin rpy="0 0 0" xyz=" 0.17 ${dir*0.19} -0.04"/>
             <axis xyz="0 0 1"/>
         </joint>
         <link name="rear_caster_wheel_${prefix}">
             <collision>
-                <origin xyz="0 0 0.0" rpy="0 ${pi/2} 0"/>
-                <geometry>
-                <cylinder length="0.02" radius="0.03"/>
-                </geometry>
-            </collision>
-            <visual>
-                <origin xyz="0 0 0.0" rpy="0 ${pi/2} 0"/>
+                <origin xyz="0 0 0.0" rpy="0 0 0"/>
+                <geometry>
+                <cylinder length="0.02" radius="0.03"/>
+                </geometry>
+            </collision>
+            <visual>
+                <origin xyz="0 0 0.0" rpy="0 0 0"/>
                 <geometry>
                 <cylinder length="0.02" radius="0.03"/>
@@ -88,5 +90,5 @@
             </visual>
             <inertial>
-                <origin xyz="0 0 0.0" rpy="0 ${pi/2} 0"/>
+                <origin xyz="0 0 0.0" rpy="0 0 0"/>
                 <mass value="0.1"/>
                 <xacro:cylinder_inertia m="0.1" r="0.03" h="0.02"/>
@@ -96,5 +98,5 @@
             <parent link="rear_caster_rotate_${prefix}"/>
             <child link="rear_caster_wheel_${prefix}"/>
-            <origin rpy="0 0 0" xyz="0 -0.02 -0.04"/>
+            <origin rpy="0 1.57 1.57" xyz="-0.02 0 -0.04"/>
             <axis xyz="1 0 0"/>
             <limit effort="1000000" velocity="20.0"/>
@@ -128,16 +130,17 @@
             <!--origin rpy="0 0 0" xyz="0.16 0.1 -0.015"/-->
             <child link="front_caster_rotate_${prefix}"/>
-            <origin rpy="0 0 0" xyz="${dir*0.19} -0.17 -0.04"/>
+            <!-- <origin rpy="0 0 0" xyz="${dir*0.19} -0.17 -0.04"/> -->
+            <origin rpy="0 0 0" xyz="-0.17 ${dir*0.19} -0.04"/>
             <axis xyz="0 0 1"/>
         </joint>
         <link name="front_caster_wheel_${prefix}">
             <collision>
-                <origin xyz="0 0 0.0" rpy="0 ${pi/2} 0"/>
-                <geometry>
-                <cylinder length="0.02" radius="0.03"/>
-                </geometry>
-            </collision>
-            <visual>
-                <origin xyz="0 0 0.0" rpy="0 ${pi/2} 0"/>
+                <origin xyz="0 0 0.0" rpy="0 0 0"/>
+                <geometry>
+                <cylinder length="0.02" radius="0.03"/>
+                </geometry>
+            </collision>
+            <visual>
+                <origin xyz="0 0 0.0" rpy="0 0 0"/>
                 <geometry>
                 <cylinder length="0.02" radius="0.03"/>
@@ -146,5 +149,5 @@
             </visual>
             <inertial>
-                <origin xyz="0 0 0.0" rpy="0 ${pi/2} 0"/>
+                <origin xyz="0 0 0.0" rpy="0 0 0"/>
                 <mass value="0.1"/>
                 <xacro:cylinder_inertia m="0.1" r="0.03" h="0.02"/>
@@ -154,6 +157,6 @@
             <parent link="front_caster_rotate_${prefix}"/>
             <child link="front_caster_wheel_${prefix}"/>
-            <origin rpy="0 0 0" xyz="0 -0.02 -0.04"/>
-            <axis xyz="1 0 0"/>
+            <origin rpy="0 1.57 1.57" xyz="-0.02 0 -0.04"/>
+            <axis xyz="0 0 1"/>
             <limit effort="1000000" velocity="20.0"/>
         </joint>
@@ -185,5 +188,5 @@
             <parent link="base_link"/>
             <child link="Wheel_${prefix}"/>
-            <origin rpy="0 1.57 3.14" xyz="${dir*0.18} 0 -0.04"/>
+            <origin rpy="0 1.57 1.57" xyz="0 ${dir*0.18} -0.04"/>
             <axis xyz="0 0 1"/>
             <limit effort="1000000" velocity="20.0"/>
@@ -251,15 +254,15 @@
         <parent link="base_link"/>
         <child link="camera_link"/>
-        <origin xyz="0.0 0.185 0.30" rpy="0 0 0"/>
+        <origin xyz="0.175 0 0.30" rpy="0 0 0"/>
     </joint>
     <link name="camera_link">
         <visual>
             <geometry>
-                <box size="-0.1 0.03 0.03"/>
+                <box size=" 0.03 0.1 0.03"/>
             </geometry>
         </visual>
         <collision>
             <geometry>
-                <box size="-0.1 0.03 0.03"/>
+                <box size=" 0.03 0.1 0.03"/>
             </geometry>
         </collision>
@@ -268,5 +271,5 @@
         <parent link="camera_link"/>
         <child link="camera_link_optical"/>
-        <origin xyz="0 0 0" rpy="0 0 ${pi/2}"/>
+        <origin xyz="0 0 0" rpy="0 0 0"/>
     </joint>
     <link name="camera_link_optical">
